File: builds/2019-07-15 chassis heater/kicad/oven-lazy.sch (KiCad schematic (older format))
At the start: 13 parts, among them Q1 TIP122, U1 LM324, U2 L7805

Commit message: fix schematic
Parts:
- removed Q1: TIP122, Package_TO_SOT_THT:TO-220-3_Vertical, symbol Transistor_BJT:TIP122
- removed U2: L7805, symbol Regulator_Linear:L7805
- added Q?: TIP122, Package_TO_SOT_THT:TO-220-3_Vertical, symbol Transistor_BJT:TIP122
- added U?: L7805, symbol Regulator_Linear:L7805
- NTC: renamed from TH1; value 10K NTC -> 10K
- renumbered RV1 to POT
Connections:
- net 12V: now also U?.1 (IN)
- net GND: now also Q?.3 (E), U?.2 (GND)
- net at R6.2, U1.2 (-): now also NTC.1, R3.2; no longer POT.2
- net at R5.1: now also Q?.1 (B)
- new net: POT.2, U1.3 (+)
- new net: Q?.2 (C), U?.3 (OUT)
Other:
- note added: "heater (running)"
- note added: "heater (startup)"
- moved on the sheet: C1, D1, D2, NTC, POT, R1, R2, R3
